Commit message: Update sence_main.xacro

File: sence_main_description/urdf/sence_main.xacro (robot description, xacro)
@@ -5,4 +5,6 @@
 <xacro:include filename="$(find sence_main_description)/urdf/sence_main.gazebo" />
 <link name="base_link">
+</link>
+<link name="core">
   <inertial>
     <origin xyz="-0.0003058772493282508 -8.555215015878667e-05 -7.892579365353808e-05" rpy="0 0 0"/>
@@ -24,3 +26,8 @@
   </collision>
 </link>
+<joint name="con" type="fixed">
+  <origin rpy="0 0 0" xyz="0 0 0"/>
+  <parent link="base_link"/>
+  <child link="core"/>
+</joint>
 </robot>
