Commit message: Comb Pybullet / RTB / Comb URDF Update
Comb Pybullet impletementation complete with movable joints. RTB tests to transfer matlab code to python toolbox. Comb URDF Update to resolve issue from not rerunning xacro.

File: sence_main_description/urdf/sence_comb.urdf (robot description, URDF)
Before this commit: robot sence_main, 18 links, 17 joints
Joints:
- joint back_left_leg_Rev1: axis 1.0 0.0 0.0 -> 1.0 0.0 -0.0; origin xyz=-0.04375 -0.00555 0.0 rpy=0 0 0 -> xyz=0.01348 0.002676 -0.038139 rpy=0 0 0
- joint back_left_leg_Rev2: origin xyz=-0.033926 0.00678 0.0002 rpy=0 0 0 -> xyz=-0.033927 0.00678 0.0002 rpy=0 0 0
- joint back_left_leg_system_connection: origin xyz=-0.20 -0.15 0 rpy=0 0 0 -> xyz=-0.1438 -0.1250 0.0381 rpy=0 0 0
- joint back_right_leg_Rev1: axis 1.0 0.0 0.0 -> 1.0 0.0 -0.0; origin xyz=-0.04375 -0.00555 0.0 rpy=0 0 0 -> xyz=0.01348 0.002676 -0.038139 rpy=0 0 0
- joint back_right_leg_Rev2: origin xyz=-0.033926 0.00678 0.0002 rpy=0 0 0 -> xyz=-0.033927 0.00678 0.0002 rpy=0 0 0
- joint back_right_leg_system_connection: origin xyz=0.20 -0.15 0 rpy=0 3.14159 0 -> xyz=0.1438 -0.1250 -0.0381 rpy=0 3.14159 0
- joint front_left_leg_Rev1: axis 1.0 0.0 0.0 -> 1.0 0.0 -0.0; origin xyz=-0.04375 -0.00555 0.0 rpy=0 0 0 -> xyz=0.01348 0.002676 -0.038139 rpy=0 0 0
- joint front_left_leg_Rev2: origin xyz=-0.033926 0.00678 0.0002 rpy=0 0 0 -> xyz=-0.033927 0.00678 0.0002 rpy=0 0 0
- joint front_left_leg_system_connection: origin xyz=-0.20 0.15 0 rpy=3.14159 0 0 -> xyz=-0.1438 0.1250 -0.0381 rpy=3.14159 0 0
- joint front_right_leg_Rev1: axis 1.0 0.0 0.0 -> 1.0 0.0 -0.0; origin xyz=-0.04375 -0.00555 0.0 rpy=0 0 0 -> xyz=0.01348 0.002676 -0.038139 rpy=0 0 0
- joint front_right_leg_Rev2: origin xyz=-0.033926 0.00678 0.0002 rpy=0 0 0 -> xyz=-0.033927 0.00678 0.0002 rpy=0 0 0
- joint front_right_leg_system_connection: origin xyz=0.20 0.15 0 rpy=3.14159 3.14159 0 -> xyz=0.1438 0.1250 0.0381 rpy=3.14159 3.14159 0
