Commit message: URDF Fix / Rviz + Joint Gui Complete
-Resolved URDF misaligned joint issues caused by double generation of URDF from
a fusion file without clearing changes from previous generation.

-Added joint_state_publisher_gui to launch files instead of joint_state_publisher
due to gui being forked to a separate package, stopping gui from launching
and causing conflict if both were active.

Logged: 9/08/2022 12:27am

File: sence_leg_description/urdf/materials.xacro (robot description, xacro)
@@ -4,3 +4,6 @@
   <color rgba="0.700 0.700 0.700 1.000"/>
 </material>
+<material name="black">
+  <color rgba="1 1 1 1"/>
+</material>
 </robot>

File: sence_leg_description/urdf/sence_leg.xacro (robot description, xacro)
@@ -6,5 +6,5 @@
 <link name="base_link">
   <inertial>
-    <origin xyz="-0.028184578381233765 0.0020392786644214244 -9.813214185615953e-06" rpy="0 0 0"/>
+    <origin xyz="0.029044932513473305 0.010265080427010284 -0.03814827760382364" rpy="0 0 0"/>
     <mass value="0.15187448298114298"/>
     <inertia ixx="5.3e-05" iyy="6.1e-05" izz="6.9e-05" ixy="-6e-06" iyz="0.0" ixz="0.0"/>
@@ -15,5 +15,5 @@
       <mesh filename="package://sence_leg_description/meshes/base_link.stl" scale="0.001 0.001 0.001"/>
     </geometry>
-    <material name="silver"/>
+    <material name="plastic_matte_black"/>
   </visual>
   <collision>
@@ -26,17 +26,17 @@
 <link name="HMMR_Leg_J2_v1_1">
   <inertial>
-    <origin xyz="-0.04078345991823647 -0.01323108575665483 0.00021630889019305232" rpy="0 0 0"/>
+    <origin xyz="-0.04078394902352935 -0.013231283994066126 0.00021684450055575039" rpy="0 0 0"/>
     <mass value="0.09734685103972182"/>
     <inertia ixx="2.2e-05" iyy="3.6e-05" izz="4e-05" ixy="-2e-06" iyz="0.0" ixz="0.0"/>
   </inertial>
   <visual>
-    <origin xyz="0.04375 0.00555 0.0" rpy="0 0 0"/>
+    <origin xyz="-0.01348 -0.002676 0.038139" rpy="0 0 0"/>
     <geometry>
       <mesh filename="package://sence_leg_description/meshes/HMMR_Leg_J2_v1_1.stl" scale="0.001 0.001 0.001"/>
     </geometry>
-    <material name="silver"/>
+    <material name="plastic_matte_black"/>
   </visual>
   <collision>
-    <origin xyz="0.04375 0.00555 0.0" rpy="0 0 0"/>
+    <origin xyz="-0.01348 -0.002676 0.038139" rpy="0 0 0"/>
     <geometry>
       <mesh filename="package://sence_leg_description/meshes/HMMR_Leg_J2_v1_1.stl" scale="0.001 0.001 0.001"/>
@@ -46,17 +46,17 @@
 <link name="HMMR_Leg_J3_v1_1">
   <inertial>
-    <origin xyz="-0.06366993215147018 -0.021943102238793904 0.0024098327148608222" rpy="0 0 0"/>
+    <origin xyz="-0.06366942125676311 -0.021943300476205383 0.0024103683252244337" rpy="0 0 0"/>
     <mass value="0.1208747488020619"/>
     <inertia ixx="3.4e-05" iyy="0.000102" izz="0.000104" ixy="1.4e-05" iyz="-1e-06" ixz="2e-06"/>
   </inertial>
   <visual>
-    <origin xyz="0.077676 -0.00123 -0.0002" rpy="0 0 0"/>
+    <origin xyz="0.020447 -0.009456 0.037939" rpy="0 0 0"/>
     <geometry>
       <mesh filename="package://sence_leg_description/meshes/HMMR_Leg_J3_v1_1.stl" scale="0.001 0.001 0.001"/>
     </geometry>
-    <material name="silver"/>
+    <material name="plastic_matte_black"/>
   </visual>
   <collision>
-    <origin xyz="0.077676 -0.00123 -0.0002" rpy="0 0 0"/>
+    <origin xyz="0.020447 -0.009456 0.037939" rpy="0 0 0"/>
     <geometry>
       <mesh filename="package://sence_leg_description/meshes/HMMR_Leg_J3_v1_1.stl" scale="0.001 0.001 0.001"/>
@@ -66,17 +66,17 @@
 <link name="HMMR_Leg_J4_1">
   <inertial>
-    <origin xyz="-0.06827232180237036 0.01066109112327507 0.02089322420417813" rpy="0 0 0"/>
+    <origin xyz="-0.06827181090766318 0.01066089288586344 0.020893759814543007" rpy="0 0 0"/>
     <mass value="0.052701725493830516"/>
     <inertia ixx="1.8e-05" iyy="7.3e-05" izz="7.2e-05" ixy="1.4e-05" iyz="0.0" ixz="-1e-06"/>
   </inertial>
   <visual>
-    <origin xyz="0.142683 0.01877 0.019275" rpy="0 0 0"/>
+    <origin xyz="0.085454 0.010544 0.057414" rpy="0 0 0"/>
     <geometry>
       <mesh filename="package://sence_leg_description/meshes/HMMR_Leg_J4_1.stl" scale="0.001 0.001 0.001"/>
     </geometry>
-    <material name="silver"/>
+    <material name="carbon_fiber_twill"/>
   </visual>
   <collision>
-    <origin xyz="0.142683 0.01877 0.019275" rpy="0 0 0"/>
+    <origin xyz="0.085454 0.010544 0.057414" rpy="0 0 0"/>
     <geometry>
       <mesh filename="package://sence_leg_description/meshes/HMMR_Leg_J4_1.stl" scale="0.001 0.001 0.001"/>
@@ -85,11 +85,11 @@
 </link>
 <joint name="Rev1" type="continuous">
-  <origin xyz="-0.04375 -0.00555 0.0" rpy="0 0 0"/>
+  <origin xyz="0.01348 0.002676 -0.038139" rpy="0 0 0"/>
   <parent link="base_link"/>
   <child link="HMMR_Leg_J2_v1_1"/>
-  <axis xyz="1.0 0.0 0.0"/>
+  <axis xyz="1.0 0.0 -0.0"/>
 </joint>
 <joint name="Rev2" type="revolute">
-  <origin xyz="-0.033926 0.00678 0.0002" rpy="0 0 0"/>
+  <origin xyz="-0.033927 0.00678 0.0002" rpy="0 0 0"/>
   <parent link="HMMR_Leg_J2_v1_1"/>
   <child link="HMMR_Leg_J3_v1_1"/>

File: sence_leg_description/urdf/sence_leg_macro.xacro (robot description, xacro)
@@ -6,5 +6,5 @@
 <link name="${prefix}base_link">
   <inertial>
-    <origin xyz="-0.028184578381233765 0.0020392786644214244 -9.813214185615953e-06" rpy="0 0 0"/>
+    <origin xyz="0.029044932513473305 0.010265080427010284 -0.03814827760382364" rpy="0 0 0"/>
     <mass value="0.15187448298114298"/>
     <inertia ixx="5.3e-05" iyy="6.1e-05" izz="6.9e-05" ixy="-6e-06" iyz="0.0" ixz="0.0"/>
@@ -26,10 +26,10 @@
 <link name="${prefix}HMMR_Leg_J2_v1_1">
   <inertial>
-    <origin xyz="-0.04078345991823647 -0.01323108575665483 0.00021630889019305232" rpy="0 0 0"/>
+    <origin xyz="-0.04078394902352935 -0.013231283994066126 0.00021684450055575039" rpy="0 0 0"/>
     <mass value="0.09734685103972182"/>
     <inertia ixx="2.2e-05" iyy="3.6e-05" izz="4e-05" ixy="-2e-06" iyz="0.0" ixz="0.0"/>
   </inertial>
   <visual>
-    <origin xyz="0.04375 0.00555 0.0" rpy="0 0 0"/>
+    <origin xyz="-0.01348 -0.002676 0.038139" rpy="0 0 0"/>
     <geometry>
       <mesh filename="package://sence_leg_description/meshes/HMMR_Leg_J2_v1_1.stl" scale="0.001 0.001 0.001"/>
@@ -38,5 +38,5 @@
   </visual>
   <collision>
-    <origin xyz="0.04375 0.00555 0.0" rpy="0 0 0"/>
+    <origin xyz="-0.01348 -0.002676 0.038139" rpy="0 0 0"/>
     <geometry>
       <mesh filename="package://sence_leg_description/meshes/HMMR_Leg_J2_v1_1.stl" scale="0.001 0.001 0.001"/>
@@ -46,10 +46,10 @@
 <link name="${prefix}HMMR_Leg_J3_v1_1">
   <inertial>
-    <origin xyz="-0.06366993215147018 -0.021943102238793904 0.0024098327148608222" rpy="0 0 0"/>
+    <origin xyz="-0.06366942125676311 -0.021943300476205383 0.0024103683252244337" rpy="0 0 0"/>
     <mass value="0.1208747488020619"/>
     <inertia ixx="3.4e-05" iyy="0.000102" izz="0.000104" ixy="1.4e-05" iyz="-1e-06" ixz="2e-06"/>
   </inertial>
   <visual>
-    <origin xyz="0.077676 -0.00123 -0.0002" rpy="0 0 0"/>
+    <origin xyz="0.020447 -0.009456 0.037939" rpy="0 0 0"/>
     <geometry>
       <mesh filename="package://sence_leg_description/meshes/HMMR_Leg_J3_v1_1.stl" scale="0.001 0.001 0.001"/>
@@ -58,5 +58,5 @@
   </visual>
   <collision>
-    <origin xyz="0.077676 -0.00123 -0.0002" rpy="0 0 0"/>
+    <origin xyz="0.020447 -0.009456 0.037939" rpy="0 0 0"/>
     <geometry>
       <mesh filename="package://sence_leg_description/meshes/HMMR_Leg_J3_v1_1.stl" scale="0.001 0.001 0.001"/>
@@ -66,10 +66,10 @@
 <link name="${prefix}HMMR_Leg_J4_1">
   <inertial>
-    <origin xyz="-0.06827232180237036 0.01066109112327507 0.02089322420417813" rpy="0 0 0"/>
+    <origin xyz="-0.06827181090766318 0.01066089288586344 0.020893759814543007" rpy="0 0 0"/>
     <mass value="0.052701725493830516"/>
     <inertia ixx="1.8e-05" iyy="7.3e-05" izz="7.2e-05" ixy="1.4e-05" iyz="0.0" ixz="-1e-06"/>
   </inertial>
   <visual>
-    <origin xyz="0.142683 0.01877 0.019275" rpy="0 0 0"/>
+    <origin xyz="0.085454 0.010544 0.057414" rpy="0 0 0"/>
     <geometry>
       <mesh filename="package://sence_leg_description/meshes/HMMR_Leg_J4_1.stl" scale="0.001 0.001 0.001"/>
@@ -78,5 +78,5 @@
   </visual>
   <collision>
-    <origin xyz="0.142683 0.01877 0.019275" rpy="0 0 0"/>
+    <origin xyz="0.085454 0.010544 0.057414" rpy="0 0 0"/>
     <geometry>
       <mesh filename="package://sence_leg_description/meshes/HMMR_Leg_J4_1.stl" scale="0.001 0.001 0.001"/>
@@ -90,11 +90,11 @@
 </joint>
 <joint name="${prefix}Rev1" type="continuous">
-  <origin xyz="-0.04375 -0.00555 0.0" rpy="0 0 0"/>
+  <origin xyz="0.01348 0.002676 -0.038139" rpy="0 0 0"/>
   <parent link="${prefix}base_link"/>
   <child link="${prefix}HMMR_Leg_J2_v1_1"/>
-  <axis xyz="1.0 0.0 0.0"/>
+  <axis xyz="1.0 0.0 -0.0"/>
 </joint>
 <joint name="${prefix}Rev2" type="revolute">
-  <origin xyz="-0.033926 0.00678 0.0002" rpy="0 0 0"/>
+  <origin xyz="-0.033927 0.00678 0.0002" rpy="0 0 0"/>
   <parent link="${prefix}HMMR_Leg_J2_v1_1"/>
   <child link="${prefix}HMMR_Leg_J3_v1_1"/>

File: sence_main_description/urdf/sence_comb.urdf (robot description, URDF)
Before this commit: robot sence_main, 17 links, 16 joints
Links:
- added link core, mass 0.866383082373337; collision mesh filename=package://sence_main_description/meshes/base_link.stl scale=0.001 0.001 0.001; visual mesh filename=package://sence_main_description/meshes/base_link.stl scale=0.001 0.001 0.001
- link base_link: mass 0.866383082373337 -> None; geometry 
Joints:
- added joint con: type fixed, parent base_link, child core, origin xyz=0 0 0 rpy=0 0 0
- joint back_left_leg_system_connection: parent base_link -> core
- joint back_right_leg_system_connection: parent base_link -> core
- joint front_left_leg_system_connection: parent base_link -> core
- joint front_right_leg_system_connection: parent base_link -> core

File: sence_main_description/urdf/sence_comb.xacro (robot description, xacro)
@@ -6,4 +6,6 @@
 <xacro:include filename="$(find sence_main_description)/urdf/sence_main.gazebo" />
 <link name="base_link">
+</link>
+<link name="core">
   <inertial>
     <origin xyz="-0.0003058772493282508 -8.555215015878667e-05 -7.892579365353808e-05" rpy="0 0 0"/>
@@ -25,7 +27,12 @@
   </collision>
 </link>
-<xacro:sence_leg_macro prefix="back_right_leg_" parent="base_link" adjT="0.20 -0.15 0" adjR="0 3.14159 0"/>
-<xacro:sence_leg_macro prefix="back_left_leg_" parent="base_link" adjT="-0.20 -0.15 0" adjR="0 0 0"/>
-<xacro:sence_leg_macro prefix="front_right_leg_" parent="base_link" adjT="0.20 0.15 0" adjR="3.14159 3.14159 0"/>
-<xacro:sence_leg_macro prefix="front_left_leg_" parent="base_link" adjT="-0.20 0.15 0" adjR="3.14159 0 0"/>
+<joint name="con" type="fixed">
+  <origin rpy="0 0 0" xyz="0 0 0"/>
+  <parent link="base_link"/>
+  <child link="core"/>
+</joint>
+<xacro:sence_leg_macro prefix="back_right_leg_" parent="core" adjT="0.1438 -0.1250 -0.0381" adjR="0 3.14159 0"/>
+<xacro:sence_leg_macro prefix="back_left_leg_" parent="core" adjT="-0.1438 -0.1250 0.0381" adjR="0 0 0"/>
+<xacro:sence_leg_macro prefix="front_right_leg_" parent="core" adjT="0.1438 0.1250 0.0381" adjR="3.14159 3.14159 0"/>
+<xacro:sence_leg_macro prefix="front_left_leg_" parent="core" adjT="-0.1438 0.1250 -0.0381" adjR="3.14159 0 0"/>
 </robot>
