Commit message: Update sence_leg.xacro

File: sence_leg_description/urdf/sence_leg.xacro (robot description, xacro)
@@ -6,5 +6,5 @@
 <link name="base_link">
   <inertial>
-    <origin xyz="0.029044932513473305 0.010265080427010284 -0.03814827760382364" rpy="0 0 0"/>
+    <origin xyz="-0.028184578381233765 0.0020392786644214244 -9.813214185615953e-06" rpy="0 0 0"/>
     <mass value="0.15187448298114298"/>
     <inertia ixx="5.3e-05" iyy="6.1e-05" izz="6.9e-05" ixy="-6e-06" iyz="0.0" ixz="0.0"/>
@@ -26,10 +26,10 @@
 <link name="HMMR_Leg_J2_v1_1">
   <inertial>
-    <origin xyz="-0.04078394902352935 -0.013231283994066126 0.00021684450055575039" rpy="0 0 0"/>
+    <origin xyz="-0.04078345991823647 -0.01323108575665483 0.00021630889019305232" rpy="0 0 0"/>
     <mass value="0.09734685103972182"/>
     <inertia ixx="2.2e-05" iyy="3.6e-05" izz="4e-05" ixy="-2e-06" iyz="0.0" ixz="0.0"/>
   </inertial>
   <visual>
-    <origin xyz="-0.01348 -0.002676 0.038139" rpy="0 0 0"/>
+    <origin xyz="0.04375 0.00555 0.0" rpy="0 0 0"/>
     <geometry>
       <mesh filename="package://sence_leg_description/meshes/HMMR_Leg_J2_v1_1.stl" scale="0.001 0.001 0.001"/>
@@ -38,5 +38,5 @@
   </visual>
   <collision>
-    <origin xyz="-0.01348 -0.002676 0.038139" rpy="0 0 0"/>
+    <origin xyz="0.04375 0.00555 0.0" rpy="0 0 0"/>
     <geometry>
       <mesh filename="package://sence_leg_description/meshes/HMMR_Leg_J2_v1_1.stl" scale="0.001 0.001 0.001"/>
@@ -46,10 +46,10 @@
 <link name="HMMR_Leg_J3_v1_1">
   <inertial>
-    <origin xyz="-0.06366942125676311 -0.021943300476205383 0.0024103683252244337" rpy="0 0 0"/>
+    <origin xyz="-0.06366993215147018 -0.021943102238793904 0.0024098327148608222" rpy="0 0 0"/>
     <mass value="0.1208747488020619"/>
     <inertia ixx="3.4e-05" iyy="0.000102" izz="0.000104" ixy="1.4e-05" iyz="-1e-06" ixz="2e-06"/>
   </inertial>
   <visual>
-    <origin xyz="0.020447 -0.009456 0.037939" rpy="0 0 0"/>
+    <origin xyz="0.077676 -0.00123 -0.0002" rpy="0 0 0"/>
     <geometry>
       <mesh filename="package://sence_leg_description/meshes/HMMR_Leg_J3_v1_1.stl" scale="0.001 0.001 0.001"/>
@@ -58,5 +58,5 @@
   </visual>
   <collision>
-    <origin xyz="0.020447 -0.009456 0.037939" rpy="0 0 0"/>
+    <origin xyz="0.077676 -0.00123 -0.0002" rpy="0 0 0"/>
     <geometry>
       <mesh filename="package://sence_leg_description/meshes/HMMR_Leg_J3_v1_1.stl" scale="0.001 0.001 0.001"/>
@@ -66,10 +66,10 @@
 <link name="HMMR_Leg_J4_1">
   <inertial>
-    <origin xyz="-0.06827181090766318 0.01066089288586344 0.020893759814543007" rpy="0 0 0"/>
+    <origin xyz="-0.06827232180237036 0.01066109112327507 0.02089322420417813" rpy="0 0 0"/>
     <mass value="0.052701725493830516"/>
     <inertia ixx="1.8e-05" iyy="7.3e-05" izz="7.2e-05" ixy="1.4e-05" iyz="0.0" ixz="-1e-06"/>
   </inertial>
   <visual>
-    <origin xyz="0.085454 0.010544 0.057414" rpy="0 0 0"/>
+    <origin xyz="0.142683 0.01877 0.019275" rpy="0 0 0"/>
     <geometry>
       <mesh filename="package://sence_leg_description/meshes/HMMR_Leg_J4_1.stl" scale="0.001 0.001 0.001"/>
@@ -78,5 +78,5 @@
   </visual>
   <collision>
-    <origin xyz="0.085454 0.010544 0.057414" rpy="0 0 0"/>
+    <origin xyz="0.142683 0.01877 0.019275" rpy="0 0 0"/>
     <geometry>
       <mesh filename="package://sence_leg_description/meshes/HMMR_Leg_J4_1.stl" scale="0.001 0.001 0.001"/>
@@ -85,11 +85,11 @@
 </link>
 <joint name="Rev1" type="continuous">
-  <origin xyz="0.01348 0.002676 -0.038139" rpy="0 0 0"/>
+  <origin xyz="-0.04375 -0.00555 0.0" rpy="0 0 0"/>
   <parent link="base_link"/>
   <child link="HMMR_Leg_J2_v1_1"/>
-  <axis xyz="1.0 0.0 -0.0"/>
+  <axis xyz="1.0 0.0 0.0"/>
 </joint>
 <joint name="Rev2" type="revolute">
-  <origin xyz="-0.033927 0.00678 0.0002" rpy="0 0 0"/>
+  <origin xyz="-0.033926 0.00678 0.0002" rpy="0 0 0"/>
   <parent link="HMMR_Leg_J2_v1_1"/>
   <child link="HMMR_Leg_J3_v1_1"/>

Commit message: Updated URDF to Revised Chassis and Legs
Updated URDF to Revised Chassis and Legs as of 04/09/2022. This Version will be used for generating and testing gaits.

File: sence_leg_description/urdf/sence_leg.xacro (robot description, xacro)
@@ -15,5 +15,5 @@
       <mesh filename="package://sence_leg_description/meshes/base_link.stl" scale="0.001 0.001 0.001"/>
     </geometry>
-    <material name="plastic_matte_black"/>
+    <material name="silver"/>
   </visual>
   <collision>
@@ -35,5 +35,5 @@
       <mesh filename="package://sence_leg_description/meshes/HMMR_Leg_J2_v1_1.stl" scale="0.001 0.001 0.001"/>
     </geometry>
-    <material name="plastic_matte_black"/>
+    <material name="silver"/>
   </visual>
   <collision>
@@ -55,5 +55,5 @@
       <mesh filename="package://sence_leg_description/meshes/HMMR_Leg_J3_v1_1.stl" scale="0.001 0.001 0.001"/>
     </geometry>
-    <material name="plastic_matte_black"/>
+    <material name="silver"/>
   </visual>
   <collision>
@@ -73,12 +73,12 @@
     <origin xyz="0.085454 0.010544 0.057414" rpy="0 0 0"/>
     <geometry>
-      <mesh filename="package://sence_leg_description/meshes/HMMR_Leg_J4_1.stl" scale="0.001 0.001 0.001"/>
+      <mesh filename="package://sence_leg_description/meshes/HMMR_Leg_J4_v1_1.stl" scale="0.001 0.001 0.001"/>
     </geometry>
-    <material name="carbon_fiber_twill"/>
+    <material name="silver"/>
   </visual>
   <collision>
     <origin xyz="0.085454 0.010544 0.057414" rpy="0 0 0"/>
     <geometry>
-      <mesh filename="package://sence_leg_description/meshes/HMMR_Leg_J4_1.stl" scale="0.001 0.001 0.001"/>
+      <mesh filename="package://sence_leg_description/meshes/HMMR_Leg_J4_v1_1.stl" scale="0.001 0.001 0.001"/>
     </geometry>
   </collision>

File: sence_leg_description/urdf/sence_leg_macro.xacro (robot description, xacro)
@@ -46,7 +46,7 @@
 <link name="${prefix}HMMR_Leg_J3_v1_1">
   <inertial>
-    <origin xyz="-0.06366942125676311 -0.021943300476205383 0.0024103683252244337" rpy="0 0 0"/>
-    <mass value="0.1208747488020619"/>
-    <inertia ixx="3.4e-05" iyy="0.000102" izz="0.000104" ixy="1.4e-05" iyz="-1e-06" ixz="2e-06"/>
+    <origin xyz="-0.05832553714381231 -0.021436456555043018 0.0024477833961314005" rpy="0 0 0"/>
+    <mass value="0.12243154933451669"/>
+    <inertia ixx="3.6e-05" iyy="9.7e-05" izz="9.9e-05" ixy="1e-05" iyz="-0.0" ixz="2e-06"/>
   </inertial>
   <visual>
@@ -65,20 +65,20 @@
 </link>
 <link name="${prefix}HMMR_Leg_J4_1">
-  <inertial>
-    <origin xyz="-0.06827181090766318 0.01066089288586344 0.020893759814543007" rpy="0 0 0"/>
-    <mass value="0.052701725493830516"/>
-    <inertia ixx="1.8e-05" iyy="7.3e-05" izz="7.2e-05" ixy="1.4e-05" iyz="0.0" ixz="-1e-06"/>
+   <inertial>
+    <origin xyz="-0.05691796302157942 0.007704167559869515 0.01964749184467182" rpy="0 0 0"/>
+    <mass value="0.05742201556545181"/>
+    <inertia ixx="2e-05" iyy="5.7e-05" izz="5.2e-05" ixy="8e-06" iyz="-0.0" ixz="1e-06"/>
   </inertial>
   <visual>
-    <origin xyz="0.085454 0.010544 0.057414" rpy="0 0 0"/>
+    <origin xyz="0.079954 0.010544 0.057414" rpy="0 0 0"/>
     <geometry>
-      <mesh filename="package://sence_leg_description/meshes/HMMR_Leg_J4_1.stl" scale="0.001 0.001 0.001"/>
+      <mesh filename="package://sence_leg_description/meshes/HMMR_Leg_J4_v1_1.stl" scale="0.001 0.001 0.001"/>
     </geometry>
     <material name="silver"/>
   </visual>
   <collision>
-    <origin xyz="0.085454 0.010544 0.057414" rpy="0 0 0"/>
+    <origin xyz="0.079954 0.010544 0.057414" rpy="0 0 0"/>
     <geometry>
-      <mesh filename="package://sence_leg_description/meshes/HMMR_Leg_J4_1.stl" scale="0.001 0.001 0.001"/>
+      <mesh filename="package://sence_leg_description/meshes/HMMR_Leg_J4_v1_1.stl" scale="0.001 0.001 0.001"/>
     </geometry>
   </collision>
@@ -103,9 +103,9 @@
 </joint>
 <joint name="${prefix}Rev3" type="revolute">
-  <origin xyz="-0.065007 -0.02 -0.019475" rpy="0 0 0"/>
+  <origin xyz="-0.059507 -0.02 -0.019475" rpy="0 0 0"/>
   <parent link="${prefix}HMMR_Leg_J3_v1_1"/>
   <child link="${prefix}HMMR_Leg_J4_1"/>
   <axis xyz="-0.0 -0.0 1.0"/>
-  <limit upper="2.356194" lower="-2.268928" effort="100" velocity="100"/>
+  <limit upper="2.094395" lower="-2.094395" effort="100" velocity="100"/>
 </joint>
 </xacro:macro>

File: sence_main_description/urdf/sence_comb.urdf (robot description, URDF)
Before this commit: robot sence_main, 18 links, 17 joints
Links:
- link back_left_leg_HMMR_Leg_J3_v1_1: mass 0.1208747488020619 -> 0.12243154933451669
- link back_left_leg_HMMR_Leg_J4_1: mass 0.052701725493830516 -> 0.05742201556545181; geometry collision mesh filename=package://sence_leg_description/meshes/HMMR_Leg_J4_v1_1.stl scale=0.001 0.001 0.001; visual mesh filename=package://sence_leg_description/meshes/HMMR_Leg_J4_v1_1.stl scale=0.001 0.001 0.001
- link back_right_leg_HMMR_Leg_J3_v1_1: mass 0.1208747488020619 -> 0.12243154933451669
- link back_right_leg_HMMR_Leg_J4_1: mass 0.052701725493830516 -> 0.05742201556545181; geometry collision mesh filename=package://sence_leg_description/meshes/HMMR_Leg_J4_v1_1.stl scale=0.001 0.001 0.001; visual mesh filename=package://sence_leg_description/meshes/HMMR_Leg_J4_v1_1.stl scale=0.001 0.001 0.001
- link core: mass 0.866383082373337 -> 0.4767252028506373
- link front_left_leg_HMMR_Leg_J3_v1_1: mass 0.1208747488020619 -> 0.12243154933451669
- link front_left_leg_HMMR_Leg_J4_1: mass 0.052701725493830516 -> 0.05742201556545181; geometry collision mesh filename=package://sence_leg_description/meshes/HMMR_Leg_J4_v1_1.stl scale=0.001 0.001 0.001; visual mesh filename=package://sence_leg_description/meshes/HMMR_Leg_J4_v1_1.stl scale=0.001 0.001 0.001
- link front_right_leg_HMMR_Leg_J3_v1_1: mass 0.1208747488020619 -> 0.12243154933451669
- link front_right_leg_HMMR_Leg_J4_1: mass 0.052701725493830516 -> 0.05742201556545181; geometry collision mesh filename=package://sence_leg_description/meshes/HMMR_Leg_J4_v1_1.stl scale=0.001 0.001 0.001; visual mesh filename=package://sence_leg_description/meshes/HMMR_Leg_J4_v1_1.stl scale=0.001 0.001 0.001
Joints:
- joint back_left_leg_Rev3: limit lower=-2.268928 upper=2.356194 effort=100 velocity=100 -> lower=-2.094395 upper=2.094395 effort=100 velocity=100; origin xyz=-0.065007 -0.02 -0.019475 rpy=0 0 0 -> xyz=-0.059507 -0.02 -0.019475 rpy=0 0 0
- joint back_left_leg_system_connection: origin xyz=-0.1438 -0.1250 0.0381 rpy=0 0 0 -> xyz=-0.0826 -0.105095 0.024316 rpy=0 0 0
- joint back_right_leg_Rev3: limit lower=-2.268928 upper=2.356194 effort=100 velocity=100 -> lower=-2.094395 upper=2.094395 effort=100 velocity=100; origin xyz=-0.065007 -0.02 -0.019475 rpy=0 0 0 -> xyz=-0.059507 -0.02 -0.019475 rpy=0 0 0
- joint back_right_leg_system_connection: origin xyz=0.1438 -0.1250 -0.0381 rpy=0 3.14159 0 -> xyz=0.0826 -0.105095 -0.05196 rpy=0 3.14159 0
- joint front_left_leg_Rev3: limit lower=-2.268928 upper=2.356194 effort=100 velocity=100 -> lower=-2.094395 upper=2.094395 effort=100 velocity=100; origin xyz=-0.065007 -0.02 -0.019475 rpy=0 0 0 -> xyz=-0.059507 -0.02 -0.019475 rpy=0 0 0
- joint front_left_leg_system_connection: origin xyz=-0.1438 0.1250 -0.0381 rpy=3.14159 0 0 -> xyz=-0.0826 0.105095 -0.05196 rpy=3.14159 0 0
- joint front_right_leg_Rev3: limit lower=-2.268928 upper=2.356194 effort=100 velocity=100 -> lower=-2.094395 upper=2.094395 effort=100 velocity=100; origin xyz=-0.065007 -0.02 -0.019475 rpy=0 0 0 -> xyz=-0.059507 -0.02 -0.019475 rpy=0 0 0
- joint front_right_leg_system_connection: origin xyz=0.1438 0.1250 0.0381 rpy=3.14159 3.14159 0 -> xyz=0.0826 0.105095 0.024316 rpy=3.14159 3.14159 0

File: sence_main_description/urdf/sence_comb.xacro (robot description, xacro)
@@ -9,7 +9,7 @@
 <link name="core">
   <inertial>
-    <origin xyz="-0.0003058772493282508 -8.555215015878667e-05 -7.892579365353808e-05" rpy="0 0 0"/>
-    <mass value="0.866383082373337"/>
-    <inertia ixx="0.012736" iyy="0.003778" izz="0.016249" ixy="-0.0" iyz="0.0" ixz="0.0"/>
+    <origin xyz="0.00021651891376084524 -0.00010528739970071409 -0.014193022646418384" rpy="0 0 0"/>
+    <mass value="0.4767252028506373"/>
+    <inertia ixx="0.003452" iyy="0.000207" izz="0.003461" ixy="3e-06" iyz="2e-06" ixz="2e-06"/>
   </inertial>
   <visual>
@@ -32,7 +32,7 @@
   <child link="core"/>
 </joint>
-<xacro:sence_leg_macro prefix="back_right_leg_" parent="core" adjT="0.1438 -0.1250 -0.0381" adjR="0 3.14159 0"/>
-<xacro:sence_leg_macro prefix="back_left_leg_" parent="core" adjT="-0.1438 -0.1250 0.0381" adjR="0 0 0"/>
-<xacro:sence_leg_macro prefix="front_right_leg_" parent="core" adjT="0.1438 0.1250 0.0381" adjR="3.14159 3.14159 0"/>
-<xacro:sence_leg_macro prefix="front_left_leg_" parent="core" adjT="-0.1438 0.1250 -0.0381" adjR="3.14159 0 0"/>
+<xacro:sence_leg_macro prefix="back_right_leg_" parent="core" adjT="0.0826 -0.105095 -0.05196" adjR="0 3.14159 0"/>
+<xacro:sence_leg_macro prefix="back_left_leg_" parent="core" adjT="-0.0826 -0.105095 0.024316" adjR="0 0 0"/>
+<xacro:sence_leg_macro prefix="front_right_leg_" parent="core" adjT="0.0826 0.105095 0.024316" adjR="3.14159 3.14159 0"/>
+<xacro:sence_leg_macro prefix="front_left_leg_" parent="core" adjT="-0.0826 0.105095 -0.05196" adjR="3.14159 0 0"/>
 </robot>

File: sence_main_description/urdf/sence_main.xacro (robot description, xacro)
@@ -7,8 +7,8 @@
 </link>
 <link name="core">
-  <inertial>
-    <origin xyz="-0.0003058772493282508 -8.555215015878667e-05 -7.892579365353808e-05" rpy="0 0 0"/>
-    <mass value="0.866383082373337"/>
-    <inertia ixx="0.012736" iyy="0.003778" izz="0.016249" ixy="-0.0" iyz="0.0" ixz="0.0"/>
+<inertial>
+    <origin xyz="0.00021651891376084524 -0.00010528739970071409 -0.014193022646418384" rpy="0 0 0"/>
+    <mass value="0.4767252028506373"/>
+    <inertia ixx="0.003452" iyy="0.000207" izz="0.003461" ixy="3e-06" iyz="2e-06" ixz="2e-06"/>
   </inertial>
   <visual>
