Commit message: messing with trajectory  controllers for the legs, probably need a custom controller

File: sence_description/urdf/common/plugins.urdf.xacro (robot description, xacro)
@@ -5,5 +5,5 @@
     <gazebo>
         <plugin name="gazebo_ros_control" filename="libgazebo_ros_control.so">
-            <robotNamespace>/</robotNamespace>
+            <robotNamespace>/sence_hw</robotNamespace>
         </plugin>
     </gazebo>

File: sence_description/urdf/parts/elbow.urdf.xacro (robot description, xacro)
@@ -9,5 +9,5 @@
             <xacro:insert_block name="origin" />
             <axis xyz="0 0 1" rpy="0 0 0" />
-            <limit upper="2" lower="-2" effort="2.5" velocity="0.2" />
+            <limit upper="2" lower="-2" effort="2.5" velocity="5.5" />
         </joint>
         <!-- elbow link -->

File: sence_description/urdf/parts/shoulder.urdf.xacro (robot description, xacro)
@@ -9,5 +9,5 @@
             <xacro:insert_block name="origin" />
             <axis xyz="0 0 1" rpy="0 0 0" />
-            <limit upper="2" lower="-2" effort="2.5" velocity="0.2" />
+            <limit upper="2" lower="-2" effort="2.5" velocity="5.5" />
         </joint>
         <!-- shoulder link -->

File: sence_description/urdf/parts/wrist.urdf.xacro (robot description, xacro)
@@ -9,5 +9,5 @@
             <xacro:insert_block name="origin" />
             <axis xyz="0 0 1" rpy="0 0 0" />
-            <limit upper="2" lower="-2" effort="2.5" velocity="0.2" />
+            <limit upper="2" lower="-2" effort="2.5" velocity="5.5" />
         </joint>
         <!-- wrist link -->
