Commit message: importing cad models for hexapod urdf, WIP

File: sence_description/urdf/assemblies/arm.urdf.xacro (robot description, xacro)
@@ -29,4 +29,5 @@
                 <geometry>
                     <box size="${collision_box_x} ${collision_box_y} ${collision_box_z}"/>
+                    <!-- <mesh filename="package://sence_description/meshes/upper_shoulder.stl"/> -->
                 </geometry>
             </collision>
@@ -43,13 +44,13 @@
         <!-- shoulder -->
         <xacro:shoulder name="${name}_shoulder" parent="${name}" >
-            <origin xyz="0 0 0.035" rpy="0 0 0" />
+            <origin xyz="0 0 -0.018396" rpy="0 0 0" />
         </xacro:shoulder>
         <!-- elbow -->
         <xacro:elbow name="${name}_elbow" parent="${name}_shoulder" >
-            <origin xyz="0 0 0.035" rpy="0 0 0" />
+            <origin xyz="0.044234 0 -0.027266" rpy="0 0 0" />
         </xacro:elbow>
         <!-- wrist -->
         <xacro:wrist name="${name}_wrist" parent="${name}_elbow" >
-            <origin xyz="0 0 0.035" rpy="0 0 0" />
+            <origin xyz="0.140 0 0" rpy="0 0 0" />
         </xacro:wrist>
     </xacro:macro>

File: sence_description/urdf/parts/elbow.urdf.xacro (robot description, xacro)
@@ -9,5 +9,5 @@
             <xacro:insert_block name="origin" />
             <axis xyz="0 0 1" rpy="0 0 0" />
-            <limit upper="2" lower="2" effort="30" velocity="0.2" />
+            <limit upper="2" lower="-2" effort="2.5" velocity="0.2" />
         </joint>
         <!-- elbow link -->
@@ -26,12 +26,13 @@
             <collision >
                 <geometry>
-                    <box size="${collision_box_x} ${collision_box_y} ${collision_box_z}"/>
+                    <!-- <box size="${collision_box_x} ${collision_box_y} ${collision_box_z}"/> -->
+                    <mesh filename="package://sence_description/meshes/elbow.stl"/>
                 </geometry>
             </collision>
             <!-- inertia -->
             <inertial>
-                <mass value="0.1" />
-                <origin xyz="0 0 0" rpy="0 0 0" />
-                <inertia ixx="0.0001" ixy="0.0" ixz="0.0" iyy="0.0001" iyz="0.0" izz="0.0001" />
+                <mass value="0.176" />
+                <origin xyz="0.05811 0.000038 -0.002579" rpy="0 0 0" />
+                <inertia ixx="0.000053794" ixy="0.000004532" ixz="0.000028675" iyy="0.000196511" iyz="-0.000000913" izz="0.000167864" />
             </inertial>
         </link>

File: sence_description/urdf/parts/shoulder.urdf.xacro (robot description, xacro)
@@ -9,5 +9,5 @@
             <xacro:insert_block name="origin" />
             <axis xyz="0 0 1" rpy="0 0 0" />
-            <limit upper="2" lower="2" effort="30" velocity="0.2" />
+            <limit upper="2" lower="-2" effort="2.5" velocity="0.2" />
         </joint>
         <!-- shoulder link -->
@@ -26,12 +26,13 @@
             <collision >
                 <geometry>
-                    <box size="${collision_box_x} ${collision_box_y} ${collision_box_z}"/>
+                    <!-- <box size="${collision_box_x} ${collision_box_y} ${collision_box_z}"/> -->
+                    <mesh filename="package://sence_description/meshes/shoulder.stl"/>
                 </geometry>
             </collision>
             <!-- inertia -->
             <inertial>
-                <mass value="0.1" />
-                <origin xyz="0 0 0" rpy="0 0 0" />
-                <inertia ixx="0.0001" ixy="0.0" ixz="0.0" iyy="0.0001" iyz="0.0" izz="0.0001" />
+                <mass value="0.129" />
+                <origin xyz="0.027347 -0.00026 -0.027655" rpy="0 0 0" />
+                <inertia ixx="0.000058575" ixy="0.000000925" ixz="0.000003174" iyy="0.000075091" iyz="0.000000209" izz="0.000045978" />
             </inertial>
         </link>

File: sence_description/urdf/parts/wrist.urdf.xacro (robot description, xacro)
@@ -9,5 +9,5 @@
             <xacro:insert_block name="origin" />
             <axis xyz="0 0 1" rpy="0 0 0" />
-            <limit upper="2" lower="2" effort="30" velocity="0.2" />
+            <limit upper="2" lower="-2" effort="2.5" velocity="0.2" />
         </joint>
         <!-- wrist link -->
@@ -26,12 +26,13 @@
             <collision >
                 <geometry>
-                    <box size="${collision_box_x} ${collision_box_y} ${collision_box_z}"/>
+                    <!-- <box size="${collision_box_x} ${collision_box_y} ${collision_box_z}"/> -->
+                    <mesh filename="package://sence_description/meshes/wrist.stl"/>
                 </geometry>
             </collision>
             <!-- inertia -->
             <inertial>
-                <mass value="0.1" />
-                <origin xyz="0 0 0" rpy="0 0 0" />
-                <inertia ixx="0.0001" ixy="0.0" ixz="0.0" iyy="0.0001" iyz="0.0" izz="0.0001" />
+                <mass value="0.074" />
+                <origin xyz="0.061081 0.000014 0.003984" rpy="0 0 0" />
+                <inertia ixx="0.000010616" ixy="0.000000044" ixz="0.0000180236" iyy="0.000429333" iyz="0.000000005" izz="0.000424345" />
             </inertial>
         </link>

File: sence_description/urdf/sence_robot.urdf.xacro (robot description, xacro)
@@ -25,9 +25,15 @@
     </xacro:body>
     <!-- arms -->
-    <xacro:arm name="arm1" parent="base_link">
-        <origin xyz="0 0 0" rpy="0 0 0" />
+    <xacro:arm name="lf" parent="base_link">
+        <origin xyz="0.076509 0.076509 0" rpy="0 0 0" />
     </xacro:arm>
-    <xacro:arm name="arm2" parent="base_link">
-        <origin xyz="0 0 0" rpy="0 0 0" />
+    <xacro:arm name="rf" parent="base_link">
+        <origin xyz="0.076509 -0.076509 0" rpy="0 0 0" />
+    </xacro:arm>
+    <xacro:arm name="lm" parent="base_link">
+        <origin xyz="0 0.1082 0" rpy="0 0 0" />
+    </xacro:arm>
+    <xacro:arm name="rm" parent="base_link">
+        <origin xyz="0 -0.1082 0" rpy="0 0 0" />
     </xacro:arm>
     <!-- attach sensor packages -->

Commit message: add body mesh and rough in inertia position

File: sence_description/urdf/assemblies/arm.urdf.xacro (robot description, xacro)
@@ -28,6 +28,6 @@
             <collision >
                 <geometry>
-                    <box size="${collision_box_x} ${collision_box_y} ${collision_box_z}"/>
-                    <!-- <mesh filename="package://sence_description/meshes/upper_shoulder.stl"/> -->
+                    <!-- <box size="${collision_box_x} ${collision_box_y} ${collision_box_z}"/> -->
+                    <mesh filename="package://sence_description/meshes/upper_shoulder.stl"/>
                 </geometry>
             </collision>
@@ -48,5 +48,5 @@
         <!-- elbow -->
         <xacro:elbow name="${name}_elbow" parent="${name}_shoulder" >
-            <origin xyz="0.044234 0 -0.027266" rpy="0 0 0" />
+            <origin xyz="0.044234 0 -0.027266" rpy="${M_PI/2} ${-M_PI/6} 0" />
         </xacro:elbow>
         <!-- wrist -->

File: sence_description/urdf/parts/elbow.urdf.xacro (robot description, xacro)
@@ -33,5 +33,5 @@
             <inertial>
                 <mass value="0.176" />
-                <origin xyz="0.05811 0.000038 -0.002579" rpy="0 0 0" />
+                <origin xyz="0.05811 -0.000038 0.002579" rpy="0 0 0" />
                 <inertia ixx="0.000053794" ixy="0.000004532" ixz="0.000028675" iyy="0.000196511" iyz="-0.000000913" izz="0.000167864" />
             </inertial>

File: sence_description/urdf/sence_robot.urdf.xacro (robot description, xacro)
@@ -3,4 +3,6 @@
     <!-- materials -->
     <xacro:include filename="$(find sence_description)/urdf/common/materials.urdf.xacro" />
+    <!-- common -->
+    <xacro:include filename="$(find sence_description)/urdf/common/math.urdf.xacro" />
     <!-- assemblies -->
     <xacro:include filename="$(find sence_description)/urdf/assemblies/arm.urdf.xacro" />
@@ -22,18 +24,24 @@
     <!-- body and base link inertia -->
     <xacro:body name="base_link_inertia" parent="base_link">
-        <origin xyz="0 0 0" rpy="0 0 0" />
+        <origin xyz="0 0 -0.0515" rpy="0 0 0" />
     </xacro:body>
     <!-- arms -->
     <xacro:arm name="lf" parent="base_link">
-        <origin xyz="0.076509 0.076509 0" rpy="0 0 0" />
+        <origin xyz="0.076509 0.076509 0" rpy="0 0 ${M_PI/4}" />
     </xacro:arm>
     <xacro:arm name="rf" parent="base_link">
-        <origin xyz="0.076509 -0.076509 0" rpy="0 0 0" />
+        <origin xyz="0.076509 -0.076509 0" rpy="0 0 ${-M_PI/4}" />
     </xacro:arm>
     <xacro:arm name="lm" parent="base_link">
-        <origin xyz="0 0.1082 0" rpy="0 0 0" />
+        <origin xyz="0 0.1082 0" rpy="0 0 ${M_PI/2}" />
     </xacro:arm>
     <xacro:arm name="rm" parent="base_link">
-        <origin xyz="0 -0.1082 0" rpy="0 0 0" />
+        <origin xyz="0 -0.1082 0" rpy="0 0 ${-M_PI/2}" />
+    </xacro:arm>
+    <xacro:arm name="lb" parent="base_link">
+        <origin xyz="-0.076509 0.076509 0" rpy="0 0 ${3*M_PI/4}" />
+    </xacro:arm>
+    <xacro:arm name="rb" parent="base_link">
+        <origin xyz="-0.076509 -0.076509 0" rpy="0 0 ${-3*M_PI/4}" />
     </xacro:arm>
     <!-- attach sensor packages -->

Commit message: playing with static poses

File: sence_description/urdf/assemblies/arm.urdf.xacro (robot description, xacro)
@@ -18,4 +18,5 @@
             <visual>
                 <geometry>
+                    <!-- <mesh filename="package://sence_description/meshes/upper_shoulder.stl"/> -->
                     <mesh filename="package://sence_description/meshes/upper_shoulder.dae"/>
                 </geometry>

File: sence_description/urdf/common/plugins.urdf.xacro (robot description, xacro)
@@ -5,5 +5,5 @@
     <gazebo>
         <plugin name="gazebo_ros_control" filename="libgazebo_ros_control.so">
-            <robotNamespace>/sence_hw</robotNamespace>
+            <robotNamespace>/</robotNamespace>
         </plugin>
     </gazebo>

File: sence_description/urdf/parts/body.urdf.xacro (robot description, xacro)
@@ -14,15 +14,19 @@
             <visual>
                 <geometry>
-                    <mesh filename="package://sence_description/meshes/body.dae"/>
+                    <mesh filename="package://sence_description/meshes/body.stl"/>
+                    <!-- <mesh filename="package://sence_description/meshes/body.dae"/> -->
                 </geometry>
                 <material name="LightGrey2"/>
             </visual>
             <!-- collision -->
-            <xacro:property name="collision_box_x" value="0.075" />
+            <xacro:property name="collision_box_x" value="0.10" />
             <xacro:property name="collision_box_y" value="0.055" />
-            <xacro:property name="collision_box_z" value="0.035" />
+            <xacro:property name="collision_box_z" value="0.08" />
             <collision >
+                <!-- the origin is higher than the mesh origin -->
+                <origin xyz="0 0 ${collision_box_z}" rpy="0 0 0" />
                 <geometry>
-                    <box size="${collision_box_x} ${collision_box_y} ${collision_box_z}"/>
+                    <!-- a sphere -->
+                    <sphere radius="${collision_box_x}"/>
                 </geometry>
             </collision>

File: sence_description/urdf/parts/elbow.urdf.xacro (robot description, xacro)
@@ -9,5 +9,5 @@
             <xacro:insert_block name="origin" />
             <axis xyz="0 0 1" rpy="0 0 0" />
-            <limit upper="2" lower="-2" effort="2.5" velocity="5.5" />
+            <limit upper="1.05" lower="-1.6" effort="2.5" velocity="5.5" />
         </joint>
         <!-- elbow link -->
@@ -16,4 +16,5 @@
             <visual>
                 <geometry>
+                    <!-- <mesh filename="package://sence_description/meshes/elbow.stl"/> -->
                     <mesh filename="package://sence_description/meshes/elbow.dae"/>
                 </geometry>

File: sence_description/urdf/parts/shoulder.urdf.xacro (robot description, xacro)
@@ -9,5 +9,5 @@
             <xacro:insert_block name="origin" />
             <axis xyz="0 0 1" rpy="0 0 0" />
-            <limit upper="2" lower="-2" effort="2.5" velocity="5.5" />
+            <limit upper="1.1" lower="-1.1" effort="2.5" velocity="5.5" />
         </joint>
         <!-- shoulder link -->
@@ -16,4 +16,5 @@
             <visual>
                 <geometry>
+                    <!-- <mesh filename="package://sence_description/meshes/shoulder.stl"/> -->
                     <mesh filename="package://sence_description/meshes/shoulder.dae"/>
                 </geometry>

File: sence_description/urdf/parts/wrist.urdf.xacro (robot description, xacro)
@@ -9,5 +9,5 @@
             <xacro:insert_block name="origin" />
             <axis xyz="0 0 1" rpy="0 0 0" />
-            <limit upper="2" lower="-2" effort="2.5" velocity="5.5" />
+            <limit upper="2.75" lower="-2.75" effort="2.5" velocity="5.5" />
         </joint>
         <!-- wrist link -->
@@ -16,4 +16,5 @@
             <visual>
                 <geometry>
+                    <!-- <mesh filename="package://sence_description/meshes/wrist.stl"/> -->
                     <mesh filename="package://sence_description/meshes/wrist.dae"/>
                 </geometry>

File: sence_description/urdf/sence_robot.urdf.xacro (robot description, xacro)
@@ -20,5 +20,5 @@
         <origin xyz="0 0 0" rpy="0 0 0" />
         <axis xyz="0 0 1" rpy="0 0 0" />
-        <limit upper="0" lower="-1" effort="1000" velocity="1000" />
+        <limit upper="-0.09" lower="-0.45" effort="1000" velocity="1000" />
     </joint>
     <!-- body and base link inertia -->
