Commit message: add body mesh

File: sence_description/urdf/parts/body.urdf.xacro (robot description, xacro)
@@ -29,5 +29,5 @@
             <!-- inertia -->
             <inertial>
-                <mass value="0.1" />
+                <mass value="1.45" />
                 <origin xyz="0 0 0" rpy="0 0 0" />
                 <inertia ixx="0.0001" ixy="0.0" ixz="0.0" iyy="0.0001" iyz="0.0" izz="0.0001" />

Commit message: testing static standing in gazebo

File: sence_description/urdf/parts/body.urdf.xacro (robot description, xacro)
@@ -33,7 +33,14 @@
             <!-- inertia -->
             <inertial>
-                <mass value="1.45" />
-                <origin xyz="0 0 0" rpy="0 0 0" />
-                <inertia ixx="0.0001" ixy="0.0" ixz="0.0" iyy="0.0001" iyz="0.0" izz="0.0001" />
+                <mass value="1.445" />
+                <origin xyz="-0.045511 -0.001077 0.087828" rpy="0 0 0" />
+                <inertia
+                    ixx="0.006654466"
+                    ixy="0.0000923443"
+                    ixz="0.004203003"
+                    iyy="0.014683403"
+                    iyz="-0.00000454"
+                    izz="0.010677966"
+                />
             </inertial>
         </link>
@@ -43,11 +50,11 @@
         </gazebo>
         <!-- gazebo physics properties -->
-        <gazebo reference="${name}">
+        <!-- <gazebo reference="${name}">
 			<mu1 value="0.8"/>
 			<mu2 value="0.8"/>
-			<kp value="10000000.0" />
-			<kd value="1.0" />
+			<kp value="1000000.0" />
+			<kd value="10.0" />
 			<fdir1 value="1 0 0"/>
-		</gazebo>
+		</gazebo> -->
     </xacro:macro>
 </robot>

File: sence_description/urdf/parts/elbow.urdf.xacro (robot description, xacro)
@@ -53,5 +53,5 @@
         </gazebo>
         <!-- gazebo physics properties -->
-        <gazebo reference="${name}">
+        <!-- <gazebo reference="${name}">
 			<mu1 value="0.8"/>
 			<mu2 value="0.8"/>
@@ -59,5 +59,5 @@
 			<kd value="1.0" />
 			<fdir1 value="1 0 0"/>
-		</gazebo>
+		</gazebo> -->
     </xacro:macro>
 </robot>

File: sence_description/urdf/parts/mx-28r.urdf.xacro (robot description, xacro)
@@ -1,5 +1,5 @@
 <?xml version="1.0"?>
 <robot xmlns:xacro="http://www.ros.org/wiki/xacro">
-    <xacro:macro name="wrist" params="name">
+    <xacro:macro name="mx-28r" params="name">
         <!-- transmission -->
         <transmission name="${name}_trans" type="SimpleTransmission">

File: sence_description/urdf/parts/shoulder.urdf.xacro (robot description, xacro)
@@ -53,11 +53,11 @@
         </gazebo>
         <!-- gazebo physics properties -->
-        <gazebo reference="${name}">
+        <!-- <gazebo reference="${name}">
 			<mu1 value="0.8"/>
 			<mu2 value="0.8"/>
-			<kp value="10000000.0" />
-			<kd value="1.0" />
+			<kp value="1000000.0" />
+			<kd value="100.0" />
 			<fdir1 value="1 0 0"/>
-		</gazebo>
+		</gazebo> -->
     </xacro:macro>
 </robot>

File: sence_description/urdf/parts/wrist.urdf.xacro (robot description, xacro)
@@ -53,11 +53,11 @@
         </gazebo>
         <!-- gazebo physics properties -->
-        <gazebo reference="${name}">
-			<mu1 value="0.8"/>
-			<mu2 value="0.8"/>
-			<kp value="10000000.0" />
-			<kd value="1.0" />
-			<fdir1 value="1 0 0"/>
-		</gazebo>
+        <!-- <gazebo reference="${name}"> -->
+			<!-- <mu1 value="0.98"/> -->
+			<!-- <mu2 value="0.98"/> -->
+			<!-- <kp value="1000000.0" /> -->
+			<!-- <kd value="100.0" /> -->
+			<!-- <fdir1 value="1 0 0"/> -->
+		<!-- </gazebo> -->
     </xacro:macro>
 </robot>
