Commit message: testing cartesian controller

File: sence_description/urdf/parts/elbow.urdf.xacro (robot description, xacro)
@@ -39,12 +39,13 @@
         </link>
         <!-- transmission -->
-        <transmission name="${name}_trans" type="SimpleTransmission">
+        <transmission name="${name}_trans">
             <type>transmission_interface/SimpleTransmission</type>
-            <actuator name="${name}_motor">
-                <mechanicalReduction>1</mechanicalReduction>
-            </actuator>
             <joint name="${name}_joint">
                 <hardwareInterface>hardware_interface/PositionJointInterface</hardwareInterface>
             </joint>
+            <actuator name="${name}_motor">
+                <mechanicalReduction>1.0</mechanicalReduction>
+                <!-- <hardwareInterface>hardware_interface/PositionJointInterface</hardwareInterface> -->
+            </actuator>
         </transmission>
         <!-- gazebo colour -->

File: sence_description/urdf/parts/mx-28r.urdf.xacro (robot description, xacro)
@@ -3,12 +3,13 @@
     <xacro:macro name="mx-28r" params="name">
         <!-- transmission -->
-        <transmission name="${name}_trans" type="SimpleTransmission">
+        <transmission name="${name}_trans">
             <type>transmission_interface/SimpleTransmission</type>
-            <actuator name="${name}_motor">
-                <mechanicalReduction>1</mechanicalReduction>
-            </actuator>
             <joint name="${name}_joint">
                 <hardwareInterface>hardware_interface/PositionJointInterface</hardwareInterface>
             </joint>
+            <actuator name="${name}_motor">
+                <mechanicalReduction>1.0</mechanicalReduction>
+                <!-- <hardwareInterface>hardware_interface/PositionJointInterface</hardwareInterface> -->
+            </actuator>
         </transmission>
     </xacro:macro>

File: sence_description/urdf/parts/shoulder.urdf.xacro (robot description, xacro)
@@ -39,12 +39,13 @@
         </link>
         <!-- transmission -->
-        <transmission name="${name}_trans" type="SimpleTransmission">
+        <transmission name="${name}_trans">
             <type>transmission_interface/SimpleTransmission</type>
-            <actuator name="${name}_motor">
-                <mechanicalReduction>1</mechanicalReduction>
-            </actuator>
             <joint name="${name}_joint">
                 <hardwareInterface>hardware_interface/PositionJointInterface</hardwareInterface>
             </joint>
+            <actuator name="${name}_motor">
+                <mechanicalReduction>1.0</mechanicalReduction>
+                <!-- <hardwareInterface>hardware_interface/PositionJointInterface</hardwareInterface> -->
+            </actuator>
         </transmission>
         <!-- gazebo colour -->

File: sence_description/urdf/parts/wrist.urdf.xacro (robot description, xacro)
@@ -38,13 +38,21 @@
             </inertial>
         </link>
+        <!-- end ground contact reference frame using a link-->
+        <link name="${name}_contact"/>
+        <joint name="${name}_contact_joint" type="fixed">
+            <parent link="${name}" />
+            <child link="${name}_contact" />
+            <origin xyz="0.193702 0 0" rpy="0 0 0" />
+        </joint>
         <!-- transmission -->
-        <transmission name="${name}_trans" type="SimpleTransmission">
+        <transmission name="${name}_trans">
             <type>transmission_interface/SimpleTransmission</type>
-            <actuator name="${name}_motor">
-                <mechanicalReduction>1</mechanicalReduction>
-            </actuator>
             <joint name="${name}_joint">
                 <hardwareInterface>hardware_interface/PositionJointInterface</hardwareInterface>
             </joint>
+            <actuator name="${name}_motor">
+                <mechanicalReduction>1.0</mechanicalReduction>
+                <!-- <hardwareInterface>hardware_interface/PositionJointInterface</hardwareInterface> -->
+            </actuator>
         </transmission>
         <!-- gazebo colour -->
