Commit message: moved meshes from quad_meshes to meshes folder

File: sence_description/urdf/quad/leg.urdf.xacro (robot description, xacro)
@@ -14,5 +14,5 @@
           <origin xyz="0 0 0" rpy="0 0 0"/>
           <geometry>
-            <mesh filename="package://sence_description/quad_meshes/base_link.stl" />
+            <mesh filename="package://sence_description/meshes/base_link.stl" />
           </geometry>
           <material name="silver"/>
@@ -21,5 +21,5 @@
           <origin xyz="0 0 0" rpy="0 0 0"/>
           <geometry>
-            <mesh filename="package://sence_description/quad_meshes/base_link.stl" />
+            <mesh filename="package://sence_description/meshes/base_link.stl" />
           </geometry>
         </collision>
@@ -34,5 +34,5 @@
           <origin xyz="-0.01348 -0.002676 0.038139" rpy="0 0 0"/>
           <geometry>
-            <mesh filename="package://sence_description/quad_meshes/HMMR_Leg_J2_v1_1.stl" />
+            <mesh filename="package://sence_description/meshes/HMMR_Leg_J2_v1_1.stl" />
           </geometry>
           <material name="silver"/>
@@ -41,5 +41,5 @@
           <origin xyz="-0.01348 -0.002676 0.038139" rpy="0 0 0"/>
           <geometry>
-            <mesh filename="package://sence_description/quad_meshes/HMMR_Leg_J2_v1_1.stl" />
+            <mesh filename="package://sence_description/meshes/HMMR_Leg_J2_v1_1.stl" />
           </geometry>
         </collision>
@@ -54,5 +54,5 @@
           <origin xyz="0.020447 -0.009456 0.037939" rpy="0 0 0"/>
           <geometry>
-            <mesh filename="package://sence_description/quad_meshes/HMMR_Leg_J3_v1_1.stl" />
+            <mesh filename="package://sence_description/meshes/HMMR_Leg_J3_v1_1.stl" />
           </geometry>
           <material name="silver"/>
@@ -61,5 +61,5 @@
           <origin xyz="0.020447 -0.009456 0.037939" rpy="0 0 0"/>
           <geometry>
-            <mesh filename="package://sence_description/quad_meshes/HMMR_Leg_J3_v1_1.stl" />
+            <mesh filename="package://sence_description/meshes/HMMR_Leg_J3_v1_1.stl" />
           </geometry>
         </collision>
@@ -74,5 +74,5 @@
           <origin xyz="0.085454 0.010544 0.057414" rpy="0 0 0"/>
           <geometry>
-            <mesh filename="package://sence_description/quad_meshes/HMMR_Leg_J4_v1_1.stl" />
+            <mesh filename="package://sence_description/meshes/HMMR_Leg_J4_v1_1.stl" />
           </geometry>
           <material name="silver"/>
@@ -81,5 +81,5 @@
           <origin xyz="0.085454 0.010544 0.057414" rpy="0 0 0"/>
           <geometry>
-            <mesh filename="package://sence_description/quad_meshes/HMMR_Leg_J4_v1_1.stl" />
+            <mesh filename="package://sence_description/meshes/HMMR_Leg_J4_v1_1.stl" />
           </geometry>
         </collision>

File: sence_description/urdf/quad/main.urdf.xacro (robot description, xacro)
@@ -15,5 +15,5 @@
       <origin xyz="0 0 0" rpy="0 0 0"/>
       <geometry>
-        <mesh filename="package://sence_description/quad_meshes/chassis.stl"/>
+        <mesh filename="package://sence_description/meshes/chassis.stl"/>
       </geometry>
       <material name="silver"/>
@@ -22,5 +22,5 @@
       <origin xyz="0 0 0" rpy="0 0 0"/>
       <geometry>
-        <mesh filename="package://sence_description/quad_meshes/chassis.stl"/>
+        <mesh filename="package://sence_description/meshes/chassis.stl"/>
       </geometry>
     </collision>
